Commit message: Gripping the cup

File: challenge_problem_1/src/system_launch/models/coke_can.urdf (robot description, URDF)
Before this commit: robot coke_can_model, 1 links, 0 joints
Links:
- link coke_can: geometry collision mesh filename=package://system_launch/models/mesh/coke_can.dae scale=0.00075 0.00075 0.00075; visual mesh filename=package://system_launch/models/mesh/coke_can.dae scale=0.00075 0.00075 0.00075
